Commit message: Complete intro task steps 1-5: description install fix, RViz display, control nodes, Gazebo Harmonic launch

File: src/intro_rover_description/urdf/intro_rover_description.urdf (robot description, URDF)
Before this commit: robot intro_rover_description, 15 links, 14 joints
Joints:
- joint bl_wheel: limit (none) -> effort=100 velocity=10
- joint br_wheel: limit (none) -> effort=100 velocity=10
- joint elbow_roll: limit (none) -> effort=100 velocity=10
- joint fl_wheel: limit (none) -> effort=100 velocity=10
- joint fr_wheel: limit (none) -> effort=100 velocity=10
- joint shoulder_yaw: limit (none) -> effort=100 velocity=10
- joint wrist_roll: limit (none) -> effort=100 velocity=10
